File: auren-kicad/HearingProbeBoard-backups/HearingProbeBoard-2024-04-24_105300/HearingProbeBoard.kicad_pcb (KiCad board)
At the start: 2 copper layers, 24 x 18 mm, 11 parts, among them J1 USB_B_Mini, J2 USB_B_Mini, J3 Speaker_1, J4 Speaker_2, J5 Speaker_1, J6 Speaker_2

Commit message: Update Silkscreen to bring board name up to date
Other:
- board text added: "Open Hearing Probe"
- board text removed: "Open Hearing Auren Probe"
