File: auren-shield/auren-shield.kicad_pcb (KiCad board)
At the start: 4 copper layers, 38 x 40 mm, 49 parts, among them J1 Headphone Out, J2 MIC In, J3 HDMI_A_Molex_208658-1001, J5 Conn_01x01, J6 Conn_01x01, P1 CONN_01X06, P2 CONN_01X06, P3 CONN_01X06, P4 CONN_01X06, P5 CONN_01X06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

Commit message: Added test point pads
Parts:
- added J4: Conn_01x02, Connector_PinSocket_2.54mm:PinSocket_1x02_P2.54mm_Vertical, F.Cu at (118.4, 48.6)
Routing:
- net /TP_1: track 0.00 -> 25.5 mm, vias 0 -> 1
- net /TP_2: track 0.00 -> 22.5 mm, vias 0 -> 1
Other:
- board text added: "TP1 TP2"
